File: OpenTama.kicad_sch (KiCad schematic)
At the start: 62 parts, among them J1 Conn_01x09, J2 Conn_01x14, J3 Conn_01x07, J4 USB_C_Receptacle_USB2.0, J5 Conn_01x14, Q1 BSS138, Q2 BSS138, Q3 BSS84, SW1 LEFT, SW2 MIDDLE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

Commit message: Converted to 1206
Parts:
- C10, C13, C14, C15, C2, C3, C5, C8, C9: footprint Capacitor_SMD:C_0402_1005Metric -> Capacitor_SMD:C_1206_3216Metric
- C11, C12, C16, C4: footprint Capacitor_SMD:C_0603_1608Metric -> Capacitor_SMD:C_1206_3216Metric
- L2: footprint Inductor_SMD:L_0402_1005Metric -> Inductor_SMD:L_1206_3216Metric
- R10, R11, R12, R13, R14, R15, R16, R17, R18, R2, R20, R21, R22, R23, R24, R8, R9: footprint Resistor_SMD:R_0402_1005Metric -> Resistor_SMD:R_1206_3216Metric
- R19, R3, R4, R5, R6, R7: footprint Resistor_SMD:R_0603_1608Metric -> Resistor_SMD:R_1206_3216Metric
